File: tesselact-hw/nrf24-xcvr.kicad_sch (KiCad schematic)
At the start: 18 parts, among them U6 NRF24L01, Y1 16MHz

Commit message: Made pcb antenna footprint
Parts:
- added AE1: Antenna_Chip, my-footprints:pcb-antenna, symbol Device:Antenna_Chip
Connections:
- net ANTENNA_OUT: now also AE1.2 (PCB_Trace)
- net GND: now also AE1.1 (FEED)
Changed lines of the file:
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@@
+    (stroke (width 0) (type default) (color 0 0 0 0))
+  )
+  (wire (pts (xy 233.68 52.07) (xy 233.68 54.61))
     (stroke (width 0) (type default) (color 0 0 0 0))
   )
@@
   )
   (wire (pts (xy 158.75 129.54) (xy 153.67 129.54))
+    (stroke (width 0) (type default) (color 0 0 0 0))
+  )
+  (wire (pts (xy 228.6 52.07) (xy 228.6 64.77))
     (stroke (width 0) (type default) (color 0 0 0 0))
   )
@@
     (pin "1")
   )
+  (symbol (lib_id "Device:Antenna_Chip") (at 231.14 49.53 0) (mirror y) (unit 1)
+    (in_bom yes) (on_board yes) (fields_autoplaced)
+    (property "Reference" "AE1" (id 0) (at 234.95 45.7199 0)
+      (effects (font (size 1.27 1.27)) (justify right))
+    )
+    (property "Value" "Antenna_Chip" (id 1) (at 234.95 48.2599 0)
+      (effects (font (size 1.27 1.27)) (justify right))
+    )
+    (property "Footprint" "my-footprints:pcb-antenna" (id 2) (at 233.68 45.085 0)
+      (effects (font (size 1.27 1.27)) hide)
+    )
+    (property "Datasheet" "~" (id 3) (at 233.68 45.085 0)
+      (effects (font (size 1.27 1.27)) hide)
+    )
+    (pin "1")
+    (pin "2")
+  )
   (symbol (lib_id "power:GND") (at 78.74 74.93 0) (unit 1)
     (in_bom yes) (on_board yes)
@@
     (pin "2")
   )
+  (symbol (lib_id "power:GND") (at 233.68 54.61 0) (unit 1)
+    (in_bom yes) (on_board yes) (fields_autoplaced)
+    (property "Reference" "#PWR0135" (id 0) (at 233.68 60.96 0)
+      (effects (font (size 1.27 1.27)) hide)
+    )
+    (property "Value" "GND" (id 1) (at 233.68 59.69 0))
+    (property "Footprint" "" (id 2) (at 233.68 54.61 0)
+      (effects (font (size 1.27 1.27)) hide)
+    )
+    (property "Datasheet" "" (id 3) (at 233.68 54.61 0)
+      (effects (font (size 1.27 1.27)) hide)
+    )
+    (pin "1")
+  )
   (symbol (lib_id "power:+3V3") (at 100.33 55.88 0) (unit 1)

Commit message: Assigned footprints and removed fuse
Parts:
- AE1: value Antenna_Chip -> PCB_Antenna
- C13: footprint (none) -> Capacitor_SMD:C_0603_1608Metric
- C14, C15, C16, C17, C18, C19, C20, C21, C22: footprint (none) -> Capacitor_SMD:C_0402_1005Metric
- C23: value 1.0p -> 1p; footprint (none) -> Capacitor_SMD:C_0402_1005Metric
- L1, L2, L3: footprint (none) -> Inductor_SMD:L_0402_1005Metric
- R8, R9: footprint (none) -> Resistor_SMD:R_0402_1005Metric
- Y1: footprint (none) -> Crystal:Crystal_SMD_3225-4Pin_3.2x2.5mm
Changed lines of the file:
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@@
       (effects (font (size 1.27 1.27)) (justify left))
     )
-    (property "Footprint" "" (id 2) (at 89.8652 44.45 0)
+    (property "Footprint" "Capacitor_SMD:C_0402_1005Metric" (id 2) (at 89.8652 44.45 0)
       (effects (font (size 1.27 1.27)) hide)
     )
@@
       (effects (font (size 1.27 1.27)) (justify left))
     )
-    (property "Value" "1.0p" (id 1) (at 232.41 73.6599 0)
-      (effects (font (size 1.27 1.27)) (justify left))
-    )
-    (property "Footprint" "" (id 2) (at 229.5652 76.2 0)
+    (property "Value" "1p" (id 1) (at 232.41 73.6599 0)
+      (effects (font (size 1.27 1.27)) (justify left))
+    )
+    (property "Footprint" "Capacitor_SMD:C_0402_1005Metric" (id 2) (at 229.5652 76.2 0)
       (effects (font (size 1.27 1.27)) hide)
     )
@@
     (property "Reference" "L2" (id 0) (at 201.93 58.42 90))
     (property "Value" "3n9" (id 1) (at 201.93 60.96 90))
-    (property "Footprint" "" (id 2) (at 201.93 64.77 0)
+    (property "Footprint" "Inductor_SMD:L_0402_1005Metric" (id 2) (at 201.93 64.77 0)
       (effects (font (size 1.27 1.27)) hide)
     )
@@
       (effects (font (size 1.27 1.27)) (justify left))
     )
-    (property "Footprint" "" (id 2) (at 209.2452 96.52 0)
+    (property "Footprint" "Capacitor_SMD:C_0402_1005Metric" (id 2) (at 209.2452 96.52 0)
       (effects (font (size 1.27 1.27)) hide)
     )
@@
       (effects (font (size 1.27 1.27)) (justify left))
     )
-    (property "Footprint" "" (id 2) (at 145.7452 135.89 0)
+    (property "Footprint" "Capacitor_SMD:C_0402_1005Metric" (id 2) (at 145.7452 135.89 0)
       (effects (font (size 1.27 1.27)) hide)
     )
@@
       (effects (font (size 1.27 1.27)) (justify left))
     )
-    (property "Footprint" "" (id 2) (at 70.8152 44.45 0)
+    (property "Footprint" "Capacitor_SMD:C_0603_1608Metric" (id 2) (at 70.8152 44.45 0)
       (effects (font (size 1.27 1.27)) hide)
     )
@@
       (effects (font (size 1.27 1.27)) (justify left))
     )
-    (property "Footprint" "" (id 2) (at 197.8152 96.52 0)
+    (property "Footprint" "Capacitor_SMD:C_0402_1005Metric" (id 2) (at 197.8152 96.52 0)
       (effects (font (size 1.27 1.27)) hide)
     )
@@
       (effects (font (size 1.27 1.27)) (justify right))
     )
-    (property "Value" "Antenna_Chip" (id 1) (at 234.95 48.2599 0)
+    (property "Value" "PCB_Antenna" (id 1) (at 234.95 48.2599 0)
       (effects (font (size 1.27 1.27)) (justify right))
     )
@@
     (property "Reference" "L3" (id 0) (at 201.93 74.93 90))
     (property "Value" "2n7" (id 1) (at 201.93 77.47 90))
-    (property "Footprint" "" (id 2) (at 201.93 80.01 0)
+    (property "Footprint" "Inductor_SMD:L_0402_1005Metric" (id 2) (at 201.93 80.01 0)
       (effects (font (size 1.27 1.27)) hide)
     )
@@
       (effects (font (size 1.27 1.27)) (justify left))
     )
-    (property "Footprint" "" (id 2) (at 80.9752 44.45 0)
+    (property "Footprint" "Capacitor_SMD:C_0402_1005Metric" (id 2) (at 80.9752 44.45 0)
       (effects (font (size 1.27 1.27)) hide)
     )
@@
     (property "Reference" "R9" (id 0) (at 153.67 106.68 90))
     (property "Value" "1M" (id 1) (at 153.67 109.22 90))
-    (property "Footprint" "" (id 2) (at 153.67 114.808 90)
+    (property "Footprint" "Resistor_SMD:R_0402_1005Metric" (id 2) (at 153.67 114.808 90)
       (effects (font (size 1.27 1.27)) hide)
     )
@@
       (effects (font (size 1.27 1.27)) (justify left))
     )
-    (property "Footprint" "" (id 2) (at 69.342 96.52 90)
+    (property "Footprint" "Resistor_SMD:R_0402_1005Metric" (id 2) (at 69.342 96.52 90)
       (effects (font (size 1.27 1.27)) hide)
     )
@@
       (effects (font (size 1.27 1.27)) (justify left))
     )
-    (property "Footprint" "" (id 2) (at 80.9752 100.33 0)
+    (property "Footprint" "Capacitor_SMD:C_0402_1005Metric" (id 2) (at 80.9752 100.33 0)
       (effects (font (size 1.27 1.27)) hide)
     )
@@
       (effects (font (size 1.27 1.27)) (justify left))
     )
-    (property "Footprint" "" (id 2) (at 98.7552 44.45 0)
+    (property "Footprint" "Capacitor_SMD:C_0402_1005Metric" (id 2) (at 98.7552 44.45 0)
       (effects (font (size 1.27 1.27)) hide)
     )
@@
       (effects (font (size 1.27 1.27)) (justify left))
     )
-    (property "Footprint" "" (id 2) (at 163.5252 135.89 0)
+    (property "Footprint" "Capacitor_SMD:C_0402_1005Metric" (id 2) (at 163.5252 135.89 0)
       (effects (font (size 1.27 1.27)) hide)
     )
@@
       (effects (font (size 1.27 1.27)) (justify left))
     )
-    (property "Footprint" "" (id 2) (at 185.42 69.85 0)
+    (property "Footprint" "Inductor_SMD:L_0402_1005Metric" (id 2) (at 185.42 69.85 0)
       (effects (font (size 1.27 1.27)) hide)
     )
@@
     (property "Reference" "Y1" (id 0) (at 166.37 120.65 0))
     (property "Value" "16MHz" (id 1) (at 167.64 123.19 0))
-    (property "Footprint" "" (id 2) (at 153.67 123.19 0)
+    (property "Footprint" "Crystal:Crystal_SMD_3225-4Pin_3.2x2.5mm" (id 2) (at 153.67 123.19 0)
       (effects (font (size 1.27 1.27)) hide)
     )
@@
     (property "Reference" "C22" (id 0) (at 218.44 57.15 90))
     (property "Value" "1p5" (id 1) (at 218.44 59.69 90))
-    (property "Footprint" "" (id 2) (at 222.25 63.8048 0)
-      (effects (font (size 1.27 1.27)) hide)
-    )
+    (property "Footprint" "Capacitor_SMD:C_0402_1005Metric" (id 2) (at 222.25 63.8048 0)
+      (effects (font (size 1.27 1.27)) hide)
+    )

Commit message: Update title block data
Other:
- title: nrf24-xcvr -> tesselact
Changed lines of the file:
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@@
   (paper "A4")
   (title_block
-    (title "nrf24-xcvr")
+    (title "tesselact")
+    (date "2022-10-13")
     (rev "0.1.0")
   )
